File: board/board.kicad_pcb (KiCad board)
At the start: 2 copper layers, 21 x 13 mm, 1 part

Commit message: initial
Parts:
- added D1: BAV99, Package_TO_SOT_SMD:SOT-23, F.Cu at (148.6, 99.5)
- added D2: BAV99, Package_TO_SOT_SMD:SOT-23, F.Cu at (152.6, 99.5)
- added D3: BAV99, Package_TO_SOT_SMD:SOT-23, F.Cu at (152.6, 96.0)
- added D4: BAV99, Package_TO_SOT_SMD:SOT-23, F.Cu at (148.6, 96.0)
- added J1: 004_BASE-T_CT, on_edge:on_edge_2x05_device, F.Cu at (140.0, 96.5)
- added J2: 013_PoE_rectified, on_edge:on_edge_2x05_host, F.Cu at (161.0, 96.5)
- LOGO1: moved to B.Cu
- moved LOGO1 2.56 mm to (152.4, 99.8), turned to 180 degrees
Routing:
- net /rectifier/-: track 0.00 -> 25.2 mm, vias 0 -> 2
- net /rectifier/+: track 0.00 -> 23.9 mm
- net Net-(J1-Pad1): track 0.00 -> 16.3 mm
- net Net-(J1-Pad9): track 0.00 -> 16.2 mm
- net Net-(J1-Pad10): track 0.00 -> 16.2 mm
- net /rectifier/CT3: track 0.00 -> 12.5 mm, vias 0 -> 1
- net /rectifier/CT2: track 0.00 -> 11.6 mm, vias 0 -> 2
- net /rectifier/CT1: track 0.00 -> 10.2 mm
- net /rectifier/CT4: track 0.00 -> 7.11 mm, vias 0 -> 1
Other:
- outline, holes or cut-outs redrawn
- board text added: "osf.004"
- board text added: "osf.013"
- board text added: "osf.b134.v1.0"
